Commit message: Fixed rotation angles. Added a mesh file for RViz, but it doesn't show up well yet so it is commented out in the URDF file.

File: urdf/pcb.urdf.xacro (robot description, xacro)
@@ -6,10 +6,7 @@
        xmlns:xacro="http://ros.org/wiki/xacro"
 >
-    <xacro:property name="pcb_x_size"   value="0.0889"/>
-    <xacro:property name="pcb_y_size"   value="0.05715"/>
-    <xacro:property name="pcb_z_size"   value="0.0254"/>
-    <xacro:property name="pcb_x_offset" value="0.005"/>
-    <xacro:property name="pcb_y_offset" value="-0.09715"/>
-    <xacro:property name="pcb_z_offset" value="0.05715"/>
+    <xacro:property name="pcb_x_size"   value="0.0254"/>
+    <xacro:property name="pcb_y_size"   value="0.0254"/>
+    <xacro:property name="pcb_z_size"   value="0.0075"/>
     <link name="pcb">
         <inertial>
@@ -18,6 +15,7 @@
         </inertial>
         <visual>
-            <origin xyz="0 0 0" rpy="0 0 0"/>
+            <origin xyz="0 0 0" rpy="3.14 0 3.14"/>
             <geometry>
+                <!--mesh filename="package://os5000/mesh/os5000.stl"/-->
                 <box size="${pcb_x_size} ${pcb_y_size} ${pcb_z_size}"/>
             </geometry>
@@ -27,4 +25,5 @@
             <origin xyz="0 0 0" rpy="0 0 0"/>
             <geometry>
+                <!--mesh filename="package://os5000/mesh/os5000.stl"/-->
                 <box size="${pcb_x_size} ${pcb_y_size} ${pcb_z_size}"/>
             </geometry>
@@ -35,5 +34,5 @@
         <parent link="base_link"/>
         <child link="pcb"/>
-        <origin xyz="${pcb_x_offset+pcb_x_size/2} ${pcb_y_offset+pcb_y_size/2} ${pcb_z_offset+pcb_z_size/2}" rpy="0 0 0"/>
+        <origin xyz="0 0 0" rpy="0 0 0"/>
     </joint>
 </robot>
