Commit message: Cleaned up xacro warnings for URDF.

File: urdf/materials.urdf.xacro (robot description, xacro)
@@ -33,6 +33,6 @@
     </material>
   </xacro:macro>
-  <xacro:macro name="material_white_alpha_0.5">
-    <material name="white_alpha_0.5">
+  <xacro:macro name="material_white_alpha_0_5">
+    <material name="white_alpha_0_5">
       <color rgba="1.0 1.0 1.0 0.5"/>
     </material>
@@ -63,11 +63,11 @@
     </material>
   </xacro:macro>
-  <xacro:macro name="material_dark_green_alpha_0.5">
-    <material name="dark_green">
+  <xacro:macro name="material_dark_green_alpha_0_5">
+    <material name="dark_green_alpha_0_5">
       <color rgba="0.0 0.39 0.0 0.5"/>
     </material>
   </xacro:macro>
-  <xacro:macro name="material_brown_alpha_0.5">
-    <material name="brown">
+  <xacro:macro name="material_brown_alpha_0_5">
+    <material name="brown_alpha_0_5">
       <color rgba="0.55 0.27 0.07 0.5"/>
     </material>
